File: hardware/rev0/nfc_rev0/analog.kicad_sch (KiCad schematic)
At the start: 11 parts, among them J3 Conn_01x02

Commit message: work
Parts:
- added L?: L, symbol Device:L
Connections:
- net GND: now also L?.1
- net at C1.1, D4.2 (A), J3.2 (Pin_2): now also L?.2
Other:
- moved on the sheet: J3
Changed lines of the file:
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@@
   (junction (at 113.03 62.23) (diameter 0) (color 0 0 0 0)
   )
-  (junction (at 27.94 54.61) (diameter 0) (color 0 0 0 0)
-  )
-  (junction (at 27.94 69.85) (diameter 0) (color 0 0 0 0)
+  (junction (at 29.21 27.94) (diameter 0) (color 0 0 0 0)
+  )
+  (junction (at 29.21 43.18) (diameter 0) (color 0 0 0 0)
   )
   (junction (at 113.03 54.61) (diameter 0) (color 0 0 0 0)
@@
   (junction (at 91.44 54.61) (diameter 0) (color 0 0 0 0)
   )
+  (junction (at 48.26 69.85) (diameter 0) (color 0 0 0 0)
+  )
+  (junction (at 48.26 54.61) (diameter 0) (color 0 0 0 0)
+  )
   (junction (at 121.92 62.23) (diameter 0) (color 0 0 0 0)
   )
   (junction (at 99.06 69.85) (diameter 0) (color 0 0 0 0)
   )
-  (polyline (pts (xy 40.64 72.39) (xy 13.97 72.39))
+  (polyline (pts (xy 41.91 45.72) (xy 15.24 45.72))
     (stroke (width 0) (type default) (color 0 0 0 0))
   )
@@
     (stroke (width 0) (type default) (color 0 0 0 0))
   )
-  (polyline (pts (xy 13.97 52.07) (xy 13.97 72.39))
-    (stroke (width 0) (type default) (color 0 0 0 0))
-  )
-  (polyline (pts (xy 40.64 52.07) (xy 13.97 52.07))
+  (polyline (pts (xy 15.24 25.4) (xy 15.24 45.72))
+    (stroke (width 0) (type default) (color 0 0 0 0))
+  )
+  (wire (pts (xy 48.26 54.61) (xy 48.26 58.42))
+    (stroke (width 0) (type default) (color 0 0 0 0))
+  )
+  (polyline (pts (xy 41.91 25.4) (xy 15.24 25.4))
     (stroke (width 0) (type default) (color 0 0 0 0))
   )
@@
     (stroke (width 0) (type default) (color 0 0 0 0))
   )
-  (wire (pts (xy 53.34 63.5) (xy 54.61 63.5))
-    (stroke (width 0) (type default) (color 0 0 0 0))
-  )
-  (wire (pts (xy 54.61 54.61) (xy 62.23 54.61))
+  (wire (pts (xy 39.37 54.61) (xy 48.26 54.61))
     (stroke (width 0) (type default) (color 0 0 0 0))
   )
@@
     (stroke (width 0) (type default) (color 0 0 0 0))
   )
-  (wire (pts (xy 27.94 69.85) (xy 27.94 66.04))
-    (stroke (width 0) (type default) (color 0 0 0 0))
-  )
-  (wire (pts (xy 54.61 60.96) (xy 54.61 54.61))
-    (stroke (width 0) (type default) (color 0 0 0 0))
-  )
-  (wire (pts (xy 27.94 69.85) (xy 38.1 69.85))
+  (wire (pts (xy 29.21 43.18) (xy 29.21 39.37))
+    (stroke (width 0) (type default) (color 0 0 0 0))
+  )
+  (wire (pts (xy 29.21 43.18) (xy 39.37 43.18))
     (stroke (width 0) (type default) (color 0 0 0 0))
   )
@@
     (stroke (width 0) (type default) (color 0 0 0 0))
   )
-  (polyline (pts (xy 40.64 72.39) (xy 40.64 52.07))
+  (polyline (pts (xy 41.91 45.72) (xy 41.91 25.4))
     (stroke (width 0) (type default) (color 0 0 0 0))
   )
@@
     (stroke (width 0) (type default) (color 0 0 0 0))
   )
+  (wire (pts (xy 48.26 69.85) (xy 62.23 69.85))
+    (stroke (width 0) (type default) (color 0 0 0 0))
+  )
+  (wire (pts (xy 39.37 54.61) (xy 39.37 60.96))
+    (stroke (width 0) (type default) (color 0 0 0 0))
+  )
+  (wire (pts (xy 48.26 54.61) (xy 62.23 54.61))
+    (stroke (width 0) (type default) (color 0 0 0 0))
+  )
   (polyline (pts (xy 81.28 52.07) (xy 81.28 72.39))
     (stroke (width 0) (type default) (color 0 0 0 0))
   )
-  (wire (pts (xy 27.94 54.61) (xy 22.86 54.61))
-    (stroke (width 0) (type default) (color 0 0 0 0))
-  )
-  (wire (pts (xy 27.94 54.61) (xy 38.1 54.61))
+  (wire (pts (xy 29.21 27.94) (xy 24.13 27.94))
+    (stroke (width 0) (type default) (color 0 0 0 0))
+  )
+  (wire (pts (xy 29.21 27.94) (xy 39.37 27.94))
     (stroke (width 0) (type default) (color 0 0 0 0))
   )
@@
     (stroke (width 0) (type default) (color 0 0 0 0))
   )
-  (wire (pts (xy 54.61 69.85) (xy 62.23 69.85))
+  (wire (pts (xy 48.26 66.04) (xy 48.26 69.85))
+    (stroke (width 0) (type default) (color 0 0 0 0))
+  )
+  (wire (pts (xy 39.37 69.85) (xy 48.26 69.85))
     (stroke (width 0) (type default) (color 0 0 0 0))
   )
@@
     (stroke (width 0) (type default) (color 0 0 0 0))
   )
-  (wire (pts (xy 54.61 63.5) (xy 54.61 69.85))
-    (stroke (width 0) (type default) (color 0 0 0 0))
-  )
   (wire (pts (xy 62.23 69.85) (xy 91.44 69.85))
     (stroke (width 0) (type default) (color 0 0 0 0))
@@
     (stroke (width 0) (type default) (color 0 0 0 0))
   )
-  (wire (pts (xy 27.94 58.42) (xy 27.94 54.61))
+  (wire (pts (xy 29.21 31.75) (xy 29.21 27.94))
     (stroke (width 0) (type default) (color 0 0 0 0))
   )
@@
     (stroke (width 0) (type default) (color 0 0 0 0))
   )
-  (wire (pts (xy 27.94 69.85) (xy 22.86 69.85))
+  (wire (pts (xy 29.21 43.18) (xy 24.13 43.18))
     (stroke (width 0) (type default) (color 0 0 0 0))
   )
@@
     (stroke (width 0) (type default) (color 0 0 0 0))
   )
-  (wire (pts (xy 53.34 60.96) (xy 54.61 60.96))
+  (wire (pts (xy 39.37 69.85) (xy 39.37 63.5))
     (stroke (width 0) (type default) (color 0 0 0 0))
   )
@@
     (stroke (width 0) (type default) (color 0 0 0 0))
   )
-  (text "Antenna P/N 1462360051" (at 13.97 72.39 0)
+  (text "Antenna P/N 1462360051" (at 15.24 45.72 0)
     (effects (font (size 1.27 1.27)) (justify left bottom))
   )
@@
     (pin "2")
   )
-  (symbol (lib_id "Device:L") (at 22.86 58.42 180) (unit 1)
+  (symbol (lib_id "Device:L") (at 24.13 31.75 180) (unit 1)
     (in_bom yes) (on_board yes) (fields_autoplaced)
-    (property "Reference" "#L_{a}1" (id 0) (at 21.59 57.1499 0)
-      (effects (font (size 1.27 1.27)) (justify left))
-    )
-    (property "Value" "1.4uH" (id 1) (at 21.59 59.6899 0)
-      (effects (font (size 1.27 1.27)) (justify left))
-    )
-    (property "Footprint" "" (id 2) (at 22.86 58.42 0)
-      (effects (font (size 1.27 1.27)) hide)
-    )
-    (property "Datasheet" "~" (id 3) (at 22.86 58.42 0)
+    (property "Reference" "#L_{a}1" (id 0) (at 22.86 30.4799 0)
+      (effects (font (size 1.27 1.27)) (justify left))
+    )
+    (property "Value" "1.4uH" (id 1) (at 22.86 33.0199 0)
+      (effects (font (size 1.27 1.27)) (justify left))
+    )
+    (property "Footprint" "" (id 2) (at 24.13 31.75 0)
+      (effects (font (size 1.27 1.27)) hide)
+    )
+    (property "Datasheet" "~" (id 3) (at 24.13 31.75 0)
       (effects (font (size 1.27 1.27)) hide)
     )
@@
     (pin "2")
   )
-  (symbol (lib_id "Device:C") (at 27.94 62.23 0) (unit 1)
+  (symbol (lib_id "Device:C") (at 29.21 35.56 0) (unit 1)
     (in_bom yes) (on_board yes) (fields_autoplaced)
-    (property "Reference" "#C_{a}1" (id 0) (at 31.75 60.9599 0)
-      (effects (font (size 1.27 1.27)) (justify left))
-    )
-    (property "Value" "0.9pF" (id 1) (at 31.75 63.4999 0)
-      (effects (font (size 1.27 1.27)) (justify left))
-    )
-    (property "Footprint" "" (id 2) (at 28.9052 66.04 0)
-      (effects (font (size 1.27 1.27)) hide)
-    )
-    (property "Datasheet" "~" (id 3) (at 27.94 62.23 0)
-      (effects (font (size 1.27 1.27)) hide)
-    )
-    (pin "1")
-    (pin "2")
-  )
-  (symbol (lib_id "Connector_Generic:Conn_01x02") (at 48.26 63.5 180) (unit 1)
+    (property "Reference" "#C_{a}1" (id 0) (at 33.02 34.2899 0)
+      (effects (font (size 1.27 1.27)) (justify left))
+    )
+    (property "Value" "0.9pF" (id 1) (at 33.02 36.8299 0)
+      (effects (font (size 1.27 1.27)) (justify left))
+    )
+    (property "Footprint" "" (id 2) (at 30.1752 39.37 0)
+      (effects (font (size 1.27 1.27)) hide)
+    )
+    (property "Datasheet" "~" (id 3) (at 29.21 35.56 0)
+      (effects (font (size 1.27 1.27)) hide)
+    )
+    (pin "1")
+    (pin "2")
+  )
+  (symbol (lib_id "Connector_Generic:Conn_01x02") (at 34.29 63.5 180) (unit 1)
     (in_bom yes) (on_board yes) (fields_autoplaced)
-    (property "Reference" "J3" (id 0) (at 48.26 54.61 0))
-    (property "Value" "Conn_01x02" (id 1) (at 48.26 57.15 0))
-    (property "Footprint" "Connector_Wire:SolderWire-1.5sqmm_1x02_P7.8mm_D1.7mm_OD3.9mm" (id 2) (at 48.26 63.5 0)
-      (effects (font (size 1.27 1.27)) hide)
-    )
-    (property "Datasheet" "~" (id 3) (at 48.26 63.5 0)
+    (property "Reference" "J3" (id 0) (at 34.29 54.61 0))
+    (property "Value" "Conn_01x02" (id 1) (at 34.29 57.15 0))
+    (property "Footprint" "Connector_Wire:SolderWire-1.5sqmm_1x02_P7.8mm_D1.7mm_OD3.9mm" (id 2) (at 34.29 63.5 0)
+      (effects (font (size 1.27 1.27)) hide)
+    )
+    (property "Datasheet" "~" (id 3) (at 34.29 63.5 0)
+      (effects (font (size 1.27 1.27)) hide)
+    )
+    (pin "1")
+    (pin "2")
+  )
+  (symbol (lib_id "Device:L") (at 48.26 62.23 180) (unit 1)
+    (in_bom yes) (on_board yes) (fields_autoplaced)
+    (property "Reference" "L?" (id 0) (at 49.53 60.9599 0)
+      (effects (font (size 1.27 1.27)) (justify right))
+    )
+    (property "Value" "L" (id 1) (at 49.53 63.4999 0)
+      (effects (font (size 1.27 1.27)) (justify right))
+    )
+    (property "Footprint" "" (id 2) (at 48.26 62.23 0)
+      (effects (font (size 1.27 1.27)) hide)
+    )
+    (property "Datasheet" "~" (id 3) (at 48.26 62.23 0)
       (effects (font (size 1.27 1.27)) hide)
     )
@@
     (pin "2")
   )
-  (symbol (lib_id "Device:R") (at 22.86 66.04 180) (unit 1)
-    (in_bom yes) (on_board yes)
-    (property "Reference" "#R_{a}1" (id 0) (at 21.59 66.04 0)
-      (effects (font (size 1.27 1.27)) (justify left))
-    )
-    (property "Value" "2.3" (id 1) (at 22.86 66.04 90))
-    (property "Footprint" "" (id 2) (at 24.638 66.04 90)
-      (effects (font (size 1.27 1.27)) hide)
-    )
-    (property "Datasheet" "~" (id 3) (at 22.86 66.04 0)
-      (effects (font (size 1.27 1.27)) hide)
-    )
+  (symbol (lib_id "Device:R") (at 24.13 39.37 180) (unit 1)
+    (in_bom yes) (on_board yes)
+    (property "Reference" "#R_{a}1" (id 0) (at 22.86 39.37 0)
+      (effects (font (size 1.27 1.27)) (justify left))
+    )
+    (property "Value" "2.3" (id 1) (at 24.13 39.37 90))
+    (property "Footprint" "" (id 2) (at 25.908 39.37 90)
+      (effects (font (size 1.27 1.27)) hide)
+    )
+    (property "Datasheet" "~" (id 3) (at 24.13 39.37 0)
+      (effects (font (size 1.27 1.27)) hide)
+    )
