File: hardware/rev0/nfc_rev0/nfc_rev0.kicad_sch (KiCad schematic)
At the start: 15 parts, among them SW1 SW_DIP_x04, U1 MB85RC64TA, U2 ATtiny804-SS

Commit message: work
Parts:
- removed D?: STATUS_LED_N, LED_SMD:LED_0805_2012Metric_Pad1.15x1.40mm_HandSolder, symbol Device:LED
- removed R?: 10k, Resistor_SMD:R_0805_2012Metric_Pad1.20x1.40mm_HandSolder, symbol Device:R
- D?: value STATUS_LED_P -> STATUS_LED_G
Other:
- moved on the sheet: D?, R?

Commit message: some change i guess
Parts:
- added D?: STATUS_LED_1, LED_SMD:LED_0805_2012Metric_Pad1.15x1.40mm_HandSolder, symbol Device:LED
- added R?: 1k, Resistor_SMD:R_0805_2012Metric_Pad1.20x1.40mm_HandSolder, symbol Device:R
- D?: value STATUS_LED_G -> STATUS_LED_2
- R?: value 10k -> 1k
Connections:
- net GND: now also R?.2
- net SCL: no longer J?.3 (Pin_3), J?.3 (Pin_3), U1.5 (SDA), U2.8 (PB1)
- net at U2.12 (PA2): now also D?.2 (A)
- new net: D?.1 (K), R?.1
- new net SDA: J?.3 (Pin_3), J?.3 (Pin_3), U1.5 (SDA), U2.8 (PB1)
Other:
- moved on the sheet: D?, R6, R?
