File: hardware/rev0/nfc_rev0/serial.kicad_sch (KiCad schematic)
At the start: 9 parts, among them J1 USB_B_Mini, SW2 SW_DPDT, U3 CH340N

Commit message: some change i guess
Parts:
- D1: footprint Package_TO_SOT_SMD:SOT-23-3 -> Diode_SMD:D_SOD-123
Changed lines of the file:
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@@
     (property "Reference" "D1" (id 0) (at 123.19 35.56 0))
     (property "Value" "D_Schottky" (id 1) (at 123.19 38.1 0))
-    (property "Footprint" "Package_TO_SOT_SMD:SOT-23-3" (id 2) (at 123.19 40.64 0)
+    (property "Footprint" "Diode_SMD:D_SOD-123" (id 2) (at 123.19 40.64 0)
       (effects (font (size 1.27 1.27)) hide)
     )
